Commit message: add gazebo

File: src/robot0_description/urdf/robot0.urdf (robot description, URDF)
Before this commit: robot robot0, 30 links, 29 joints
Links:
- added link base_footprint
Joints:
- added joint base_footprint_joint: type fixed, parent base_footprint, child base_link, origin xyz=0 0 0.06 rpy=0 0 0

Commit message: fix gazebo and fix model 3d

File: src/robot0_description/urdf/robot0.urdf (robot description, URDF)
Before this commit: robot robot0, 31 links, 30 joints
Links:
- removed link 1
- removed link 2
- removed link 3
- removed link 4
- removed link 8
- link 17: geometry collision mesh filename=package://robot0_description/meshes/DC12JGB37-520_3.STL; visual mesh filename=package://robot0_description/meshes/DC12JGB37-520_3.STL
- link 5: geometry collision mesh filename=package://robot0_description/meshes/DC12JGB37-520_1.STL; visual mesh filename=package://robot0_description/meshes/DC12JGB37-520_1.STL
- link W_FR: geometry collision mesh filename=package://robot0_description/meshes/W_Right.STL; visual mesh filename=package://robot0_description/meshes/W_Right.STL
- link W_RL: geometry collision mesh filename=package://robot0_description/meshes/W_Right.STL; visual mesh filename=package://robot0_description/meshes/W_Right.STL
- link W_RR: geometry collision mesh filename=package://robot0_description/meshes/W_FL.STL; visual mesh filename=package://robot0_description/meshes/W_FL.STL
Joints:
- removed joint 1
- removed joint 10
- removed joint 11
- removed joint 12
- removed joint 13
- removed joint 14
- removed joint 15
- removed joint 16
- removed joint 17
- removed joint 18
- removed joint 19
- removed joint 2
- removed joint 20
- removed joint 21
- removed joint 22
- removed joint 23
- removed joint 3
- removed joint 4
- removed joint 5
- removed joint 6
- removed joint 7
- removed joint 8
- removed joint 9
- removed joint Tayf_nang
- removed joint W_FL
- removed joint W_FR
- removed joint W_RL
- removed joint W_RR
- removed joint cam
- added joint joint_10: type fixed, parent base_link, child 10, origin xyz=0.065771576273727 0.137279512977855 0.00823406193389999 rpy=1.5707963267949 0 -1.72157870312163, axis 0 0 0
- added joint joint_11: type fixed, parent base_link, child 11, origin xyz=0.008271576273727 0.137279512977855 0.046010455529876 rpy=1.5707963267949 0 -1.42001395046816, axis 0 0 0
- added joint joint_12: type fixed, parent base_link, child 12, origin xyz=0.008271576273728 0.137279512977854 0.2682340619339 rpy=1.5707963267949 0 0, axis 0 0 0
- added joint joint_13: type fixed, parent base_link, child 13, origin xyz=0.008271576273728 0.137279512977854 0.2782340619339 rpy=1.5707963267949 1.5707963267949 0, axis 0 0 0
- added joint joint_14: type fixed, parent base_link, child 14, origin xyz=0.008271576273728 0.128279512977855 0.2797340619339 rpy=-1.5707963267949 -0.897413987985829 3.14159265358979, axis 0 0 0
- added joint joint_15: type fixed, parent base_link, child 15, origin xyz=0.00855214883354 0.171779512977855 -0.00156454447012401 rpy=-1.5707963267949 0 0, axis 0 0 0
- added joint joint_16: type fixed, parent base_link, child 16, origin xyz=0.128271576273727 0.109279512977855 -0.0307659380661 rpy=1.5707963267949 0 1.5707963267949, axis 0 0 0
- added joint joint_17: type fixed, parent base_link, child 17, origin xyz=-0.111728423726273 0.109279512977855 -0.0307659380661 rpy=-1.5707963267949 0 -1.5707963267949, axis 0 0 0
- added joint joint_18: type fixed, parent base_link, child 18, origin xyz=0.128271576273727 -0.090720487022144 -0.0307659380661 rpy=1.5707963267949 0 1.5707963267949, axis 0 0 0
- added joint joint_19: type fixed, parent base_link, child 19, origin xyz=-0.111728423726273 -0.090720487022144 -0.0307659380661 rpy=-1.5707963267949 0 -1.5707963267949, axis 0 0 0
- added joint joint_20: type fixed, parent base_link, child 20, origin xyz=0.131271576273728 0.129279512977854 -0.00376593806610101 rpy=-1.5707963267949 0 3.14159265358979, axis 0 0 0
- added joint joint_21: type fixed, parent base_link, child 21, origin xyz=-0.114728423726273 0.089279512977854 -0.00376593806610101 rpy=-1.5707963267949 0 0, axis 0 0 0
- added joint joint_22: type fixed, parent base_link, child 22, origin xyz=0.131271576273728 -0.070720487022142 -0.003765938066101 rpy=-1.5707963267949 0 3.14159265358979, axis 0 0 0
- added joint joint_23: type fixed, parent base_link, child 23, origin xyz=-0.114728423726274 -0.115720487022144 -0.00376593806610199 rpy=-1.57079632679489 0 0, axis 0 0 0
- added joint joint_5: type fixed, parent base_link, child 5, origin xyz=0.008271576273727 0.119779512977854 0.0292340619339 rpy=-1.5707963267949 0 0, axis 0 0 0
- added joint joint_6: type fixed, parent base_link, child 6, origin xyz=0.008271576273727 0.137279512977854 0.00223406193389999 rpy=1.5707963267949 0 0, axis 0 0 0
- added joint joint_7: type fixed, parent base_link, child 7, origin xyz=0.008271576273727 0.137279512977855 0.036010455529876 rpy=1.5707963267949 0 0, axis 0 0 0
- added joint joint_9: type fixed, parent base_link, child 9, origin xyz=0.00855214883354 0.171779512977855 -0.00156454447012401 rpy=-1.5707963267949 0 0, axis 0 0 0
- added joint joint_Tayf_nang: type fixed, parent base_link, child Tayf_nang, origin xyz=0.008271576273727 0.137279512977855 0.036010455529876 rpy=1.5707963267949 0 0, axis 0 0 0
- added joint joint_W_FL: type continuous, parent base_link, child W_FL, origin xyz=-0.145628423726273 0.109279512977855 -0.0237659380661 rpy=1.5707963267949 -1.5707963267949 0, axis 0 1 0, limit effort=10.0 velocity=20.0
- added joint joint_W_FR: type continuous, parent base_link, child W_FR, origin xyz=0.162171576273727 0.109279512977855 -0.023933876070515 rpy=1.5707963267949 -1.5707963267949 0, axis 0 1 0, limit effort=10.0 velocity=20.0
- added joint joint_W_RL: type continuous, parent base_link, child W_RL, origin xyz=-0.145628423726273 -0.090720487022145 -0.023933876070516 rpy=1.5707963267949 1.5707963267949 0, axis 0 1 0, limit effort=10.0 velocity=20.0
- added joint joint_W_RR: type continuous, parent base_link, child W_RR, origin xyz=0.162171576273727 -0.090720487022145 -0.023765938066099 rpy=1.5707963267949 1.5707963267949 0, axis 0 1 0, limit effort=10.0 velocity=20.0
- added joint joint_cam: type fixed, parent base_link, child cam, origin xyz=0.008271576273727 0.173113089759183 0.338814309541528 rpy=2.57641039979753 0 0, axis 0 0 0

Commit message: fix model 3d

File: src/robot0_description/urdf/robot0.urdf (robot description, URDF)
Before this commit: robot robot0, 26 links, 25 joints
Links:
- removed link 10
- removed link 11
- removed link 12
- removed link 13
- removed link 14
- removed link 15
- removed link 16
- removed link 17
- removed link 18
- removed link 19
- removed link 20
- removed link 21
- removed link 22
- removed link 23
- removed link 5
- removed link 6
- removed link 7
- removed link 9
- removed link Tayf_nang
- removed link W_FL
- removed link W_FR
- removed link W_RL
- removed link W_RR
- removed link cam
- added link lift_arm_link, mass 0.161814335334686; collision mesh filename=package://robot0_description/meshes/lift_arm.stl; visual mesh filename=package://robot0_description/meshes/lift_arm.stl
- added link lift_base_link, mass 0.08253622186955; collision mesh filename=package://robot0_description/meshes/lift_base.stl; visual mesh filename=package://robot0_description/meshes/lift_base.stl
- added link lift_belt_link, mass 0.00663238934211694; collision mesh filename=package://robot0_description/meshes/lift_belt.stl; visual mesh filename=package://robot0_description/meshes/lift_belt.stl
- added link lift_motor_link, mass 0.0162866417907391; collision mesh filename=package://robot0_description/meshes/motor_jgb37_520_right.s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; visual mesh filename=package://robot0_description/meshes/motor_jgb37_520_right.s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
- added link lift_pipe_1_link, mass 0.0969809652163169; collision mesh filename=package://robot0_description/meshes/lift_pipe_1.stl; visual mesh filename=package://robot0_description/meshes/lift_pipe_1.stl
- added link lift_pipe_2_link, mass 0.0969809652163169; collision mesh filename=package://robot0_description/meshes/lift_pipe_2.stl; visual mesh filename=package://robot0_description/meshes/lift_pipe_2.stl
- added link lift_pulley_link, mass 0.00161689436550568; collision mesh filename=package://robot0_description/meshes/lift_pulley_20t.stl; visual mesh filename=package://robot0_description/meshes/lift_pulley_20t.stl
- added link lift_top_cap_link, mass 0.0876963777563386; collision mesh filename=package://robot0_description/meshes/lift_top_cap.stl; visual mesh filename=package://robot0_description/meshes/lift_top_cap.stl
- added link wheel_bracket_fl_link, mass 0.0210848931196573; collision mesh filename=package://robot0_description/meshes/motor_bracket_fl.stl; visual mesh filename=package://robot0_description/meshes/motor_bracket_fl.stl
- added link wheel_bracket_fr_link, mass 0.0210848931196573; collision mesh filename=package://robot0_description/meshes/motor_bracket_fr.stl; visual mesh filename=package://robot0_description/meshes/motor_bracket_fr.stl
- added link wheel_bracket_rl_link, mass 0.0210848931196573; collision mesh filename=package://robot0_description/meshes/motor_bracket_rl.stl; visual mesh filename=package://robot0_description/meshes/motor_bracket_rl.stl
- added link wheel_bracket_rr_link, mass 0.0210848931196573; collision mesh filename=package://robot0_description/meshes/motor_bracket_rr.stl; visual mesh filename=package://robot0_description/meshes/motor_bracket_rr.stl
- added link wheel_fl_link, mass 0.13187; collision mesh filename=package://robot0_description/meshes/wheel_left.stl; visual mesh filename=package://robot0_description/meshes/wheel_left.stl
- added link wheel_fr_link, mass 0.13187; collision mesh filename=package://robot0_description/meshes/wheel_right.stl; visual mesh filename=package://robot0_description/meshes/wheel_right.stl
- added link wheel_motor_fl_link, mass 0.0162866417907391; collision mesh filename=package://robot0_description/meshes/motor_jgb37_520_left.stl; visual mesh filename=package://robot0_description/meshes/motor_jgb37_520_left.stl
- added link wheel_motor_fr_link, mass 0.0162866417907391; collision mesh filename=package://robot0_description/meshes/motor_jgb37_520_right.s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; visual mesh filename=package://robot0_description/meshes/motor_jgb37_520_right.s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
- added link wheel_motor_rl_link, mass 0.0162866417907391; collision mesh filename=package://robot0_description/meshes/motor_jgb37_520_left.stl; visual mesh filename=package://robot0_description/meshes/motor_jgb37_520_left.stl
- added link wheel_motor_rr_link, mass 0.0162866417907391; collision mesh filename=package://robot0_description/meshes/motor_jgb37_520_right.s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; visual mesh filename=package://robot0_description/meshes/motor_jgb37_520_right.s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
- added link wheel_rl_link, mass 0.13187; collision mesh filename=package://robot0_description/meshes/wheel_right.stl; visual mesh filename=package://robot0_description/meshes/wheel_right.stl
- added link wheel_rr_link, mass 0.13187; collision mesh filename=package://robot0_description/meshes/wheel_left.stl; visual mesh filename=package://robot0_description/meshes/wheel_left.stl
- link base_link: mass 1.35226802643247 -> 1.352268; geometry collision mesh filename=package://robot0_description/meshes/base_link.stl; visual mesh filename=package://robot0_description/meshes/base_link.stl
Joints:
- removed joint joint_10
- removed joint joint_11
- removed joint joint_12
- removed joint joint_13
- removed joint joint_14
- removed joint joint_15
- removed joint joint_16
- removed joint joint_17
- removed joint joint_18
- removed joint joint_19
- removed joint joint_20
- removed joint joint_21
- removed joint joint_22
- removed joint joint_23
- removed joint joint_5
- removed joint joint_6
- removed joint joint_7
- removed joint joint_9
- removed joint joint_Tayf_nang
- removed joint joint_W_FL
- removed joint joint_W_FR
- removed joint joint_W_RL
- removed joint joint_W_RR
- removed joint joint_cam
- added joint lift_arm_joint: type prismatic, parent base_link, child lift_arm_link, origin xyz=0.008271576273727 0.137279512977855 0.036010455529876 rpy=1.5707963267949 0 0, axis 0 1 0, limit lower=0.0 upper=0.18 effort=100.0 velocity=0.2
- added joint lift_base_joint: type fixed, parent base_link, child lift_base_link, origin xyz=0.008271576273727 0.137279512977854 0.00223406193389999 rpy=1.5707963267949 0 0, axis 0 0 0
- added joint lift_belt_joint: type fixed, parent base_link, child lift_belt_link, origin xyz=0.008271576273728 0.128279512977855 0.2782340619339 rpy=1.5707963267949 1.5707963267949 0, axis 0 0 0
- added joint lift_motor_joint: type fixed, parent base_link, child lift_motor_link, origin xyz=0.008271576273727 0.119779512977854 0.0292340619339 rpy=-1.5707963267949 0 0, axis 0 0 0
- added joint lift_pipe_1_joint: type fixed, parent base_link, child lift_pipe_1_link, origin xyz=0.065771576273727 0.137279512977855 0.00823406193389999 rpy=1.5707963267949 0 -1.72157870312163, axis 0 0 0
- added joint lift_pipe_2_joint: type fixed, parent base_link, child lift_pipe_2_link, origin xyz=0.008271576273727 0.137279512977855 0.046010455529876 rpy=1.5707963267949 0 -1.42001395046816, axis 0 0 0
- added joint lift_pulley_joint: type fixed, parent base_link, child lift_pulley_link, origin xyz=0.008271576273728 0.128279512977855 0.2797340619339 rpy=-1.5707963267949 -0.897413987985829 3.14159265358979, axis 0 0 0
- added joint lift_top_cap_joint: type fixed, parent base_link, child lift_top_cap_link, origin xyz=0.008271576273728 0.137279512977854 0.2682340619339 rpy=1.5707963267949 0 0, axis 0 0 0
- added joint wheel_bracket_fl_joint: type fixed, parent base_link, child wheel_bracket_fl_link, origin xyz=-0.114728423726273 0.089279512977854 -0.00376593806610101 rpy=-1.5707963267949 0 0, axis 0 0 0
- added joint wheel_bracket_fr_joint: type fixed, parent base_link, child wheel_bracket_fr_link, origin xyz=0.131271576273728 0.129279512977854 -0.00376593806610101 rpy=-1.5707963267949 0 3.14159265358979, axis 0 0 0
- added joint wheel_bracket_rl_joint: type fixed, parent base_link, child wheel_bracket_rl_link, origin xyz=-0.114728423726274 -0.115720487022144 -0.00376593806610199 rpy=-1.57079632679489 0 0, axis 0 0 0
- added joint wheel_bracket_rr_joint: type fixed, parent base_link, child wheel_bracket_rr_link, origin xyz=0.131271576273728 -0.070720487022142 -0.003765938066101 rpy=-1.5707963267949 0 3.14159265358979, axis 0 0 0
- added joint wheel_fl_joint: type continuous, parent base_link, child wheel_fl_link, origin xyz=-0.145628423726273 0.109279512977855 -0.0237659380661 rpy=1.5707963267949 -1.5707963267949 0, axis 0 1 0, limit effort=10.0 velocity=20.0
- added joint wheel_fr_joint: type continuous, parent base_link, child wheel_fr_link, origin xyz=0.162171576273727 0.109279512977855 -0.023933876070515 rpy=1.5707963267949 -1.5707963267949 0, axis 0 1 0, limit effort=10.0 velocity=20.0
- added joint wheel_motor_fl_joint: type fixed, parent base_link, child wheel_motor_fl_link, origin xyz=-0.111728423726273 0.109279512977855 -0.0307659380661 rpy=-1.5707963267949 0 -1.5707963267949, axis 0 0 0
- added joint wheel_motor_fr_joint: type fixed, parent base_link, child wheel_motor_fr_link, origin xyz=0.128271576273727 0.109279512977855 -0.0307659380661 rpy=1.5707963267949 0 1.5707963267949, axis 0 0 0
- added joint wheel_motor_rl_joint: type fixed, parent base_link, child wheel_motor_rl_link, origin xyz=-0.111728423726273 -0.090720487022144 -0.0307659380661 rpy=-1.5707963267949 0 -1.5707963267949, axis 0 0 0
- added joint wheel_motor_rr_joint: type fixed, parent base_link, child wheel_motor_rr_link, origin xyz=0.128271576273727 -0.090720487022144 -0.0307659380661 rpy=1.5707963267949 0 1.5707963267949, axis 0 0 0
- added joint wheel_rl_joint: type continuous, parent base_link, child wheel_rl_link, origin xyz=-0.145628423726273 -0.090720487022145 -0.023933876070516 rpy=1.5707963267949 1.5707963267949 0, axis 0 -1 0, limit effort=10.0 velocity=20.0
- added joint wheel_rr_joint: type continuous, parent base_link, child wheel_rr_link, origin xyz=0.162171576273727 -0.090720487022145 -0.023765938066099 rpy=1.5707963267949 1.5707963267949 0, axis 0 -1 0, limit effort=10.0 velocity=20.0

Commit message: make up model in rviz

File: src/robot0_description/urdf/robot0.urdf (robot description, URDF)
Before this commit: robot robot0, 22 links, 21 joints
Links:
- removed link lift_base_link
- removed link lift_belt_link
- removed link lift_motor_link
- removed link lift_pipe_1_link
- removed link lift_pipe_2_link
- removed link lift_pulley_link
- removed link lift_top_cap_link
- removed link wheel_bracket_fl_link
- removed link wheel_bracket_fr_link
- removed link wheel_bracket_rl_link
- removed link wheel_bracket_rr_link
- removed link wheel_motor_fl_link
- removed link wheel_motor_fr_link
- removed link wheel_motor_rl_link
- removed link wheel_motor_rr_link
- link base_link: mass 1.352268 -> 1.85; geometry collision mesh filename=package://robot0_description/meshes/base_link.stl; visual mesh filename=package://robot0_description/meshes/base_link.stl
Joints:
- removed joint lift_base_joint
- removed joint lift_belt_joint
- removed joint lift_motor_joint
- removed joint lift_pipe_1_joint
- removed joint lift_pipe_2_joint
- removed joint lift_pulley_joint
- removed joint lift_top_cap_joint
- removed joint wheel_bracket_fl_joint
- removed joint wheel_bracket_fr_joint
- removed joint wheel_bracket_rl_joint
- removed joint wheel_bracket_rr_joint
- removed joint wheel_motor_fl_joint
- removed joint wheel_motor_fr_joint
- removed joint wheel_motor_rl_joint
- removed joint wheel_motor_rr_joint
- joint lift_arm_joint: axis 0 1 0 -> 0 0 1; origin xyz=0.008271576273727 0.137279512977855 0.036010455529876 rpy=1.5707963267949 0 0 -> xyz=0.008271576273727 0.137279512977855 0.036010455529876 rpy=0 0 0
- joint wheel_fr_joint: axis 0 1 0 -> 0 -1 0; origin xyz=0.162171576273727 0.109279512977855 -0.023933876070515 rpy=1.5707963267949 -1.5707963267949 0 -> xyz=0.162171576273727 0.109279512977855 -0.023933876070515 rpy=-1.5707963267949 -1.5707963267949 0
- joint wheel_rl_joint: axis 0 -1 0 -> 0 1 0; origin xyz=-0.145628423726273 -0.090720487022145 -0.023933876070516 rpy=1.5707963267949 1.5707963267949 0 -> xyz=-0.145628423726273 -0.090720487022145 -0.023933876070516 rpy=1.5707963267949 -1.5707963267949 0
- joint wheel_rr_joint: origin xyz=0.162171576273727 -0.090720487022145 -0.023765938066099 rpy=1.5707963267949 1.5707963267949 0 -> xyz=0.162171576273727 -0.090720487022145 -0.023765938066099 rpy=-1.5707963267949 -1.5707963267949 0

Commit message: use Kinematic VelocityControl to fix mecanum

File: src/robot0_description/urdf/robot0.urdf (robot description, URDF)
Before this commit: robot robot0, 7 links, 6 joints
Joints:
- joint base_footprint_joint: origin xyz=0 0 0.06 rpy=0 0 0 -> xyz=0 0 0.06 rpy=0 0 -1.5707963267948966

Commit message: improve wheel visual and joy control

File: src/robot0_description/urdf/robot0.urdf (robot description, URDF)
Before this commit: robot robot0, 7 links, 6 joints
Links:
- link wheel_fl_link: geometry collision cylinder length=0.045 radius=0.0487; visual mesh filename=package://robot0_description/meshes/wheel_left.stl
- link wheel_fr_link: geometry collision cylinder length=0.045 radius=0.0487; visual mesh filename=package://robot0_description/meshes/wheel_right.stl
- link wheel_rl_link: geometry collision cylinder length=0.045 radius=0.0487; visual mesh filename=package://robot0_description/meshes/wheel_right.stl
- link wheel_rr_link: geometry collision cylinder length=0.045 radius=0.0487; visual mesh filename=package://robot0_description/meshes/wheel_left.stl
Joints:
- joint wheel_fl_joint: origin xyz=-0.145628423726273 0.109279512977855 -0.0237659380661 rpy=1.5707963267949 -1.5707963267949 0 -> xyz=-0.145628423726273 0.109279512977855 -0.02385 rpy=1.5707963267949 -1.5707963267949 0
- joint wheel_fr_joint: origin xyz=0.162171576273727 0.109279512977855 -0.023933876070515 rpy=-1.5707963267949 -1.5707963267949 0 -> xyz=0.162171576273727 0.109279512977855 -0.02385 rpy=-1.5707963267949 -1.5707963267949 0
- joint wheel_rl_joint: origin xyz=-0.145628423726273 -0.090720487022145 -0.023933876070516 rpy=1.5707963267949 -1.5707963267949 0 -> xyz=-0.145628423726273 -0.090720487022145 -0.02385 rpy=1.5707963267949 -1.5707963267949 0
- joint wheel_rr_joint: origin xyz=0.162171576273727 -0.090720487022145 -0.023765938066099 rpy=-1.5707963267949 -1.5707963267949 0 -> xyz=0.162171576273727 -0.090720487022145 -0.02385 rpy=-1.5707963267949 -1.5707963267949 0

Commit message: add camera

File: src/robot0_description/urdf/robot0.urdf (robot description, URDF)
Before this commit: robot robot0, 7 links, 6 joints
Links:
- added link camera_link, mass 0.001
- added link camera_optical_link
Joints:
- added joint camera_joint: type fixed, parent base_link, child camera_link, origin xyz=0.00767 0.1788 0.272 rpy=0 0 1.5707963267948966
- added joint camera_optical_joint: type fixed, parent camera_link, child camera_optical_link, origin xyz=0 0 0 rpy=-1.5707963267948966 0 -1.5707963267948966

Commit message: fix physic

File: src/robot0_description/urdf/robot0.urdf (robot description, URDF)
Before this commit: robot robot0, 9 links, 8 joints
Links:
- link base_link: geometry collision box size=0.24 0.28 0.06; visual mesh filename=package://robot0_description/meshes/base_link.stl
- link lift_arm_link: geometry collision box size=0.15 0.17 0.10; visual mesh filename=package://robot0_description/meshes/lift_arm.stl

Commit message: edit camera to wide-angle camera

File: src/robot0_description/urdf/robot0.urdf (robot description, URDF)
Before this commit: robot robot0, 9 links, 8 joints
Joints:
- joint camera_joint: origin xyz=0.00767 0.1788 0.272 rpy=0 0 1.5707963267948966 -> xyz=0.00767 0.1788 0.272 rpy=0 0.5 1.5707963267948966

Commit message: add arena

File: src/robot0_description/urdf/robot0.urdf (robot description, URDF)
Before this commit: robot robot0, 9 links, 8 joints
Links:
- link lift_arm_link: geometry collision box size=0.018 0.115 0.006; collision box size=0.018 0.115 0.006
Joints:
- joint camera_joint: origin xyz=0.00767 0.1788 0.272 rpy=0 0.5 1.5707963267948966 -> xyz=0.00767 0.1788 0.272 rpy=0 0.7 1.5707963267948966

Commit message: robot modle

File: src/robot0_description/urdf/robot0.urdf (robot description, URDF)
Before this commit: robot robot0, 9 links, 8 joints
Links:
- link lift_arm_link: geometry collision box size=0.018 0.115 0.003; collision box size=0.018 0.115 0.003
Joints:
- joint lift_arm_joint: limit lower=0.0 upper=0.18 effort=100.0 velocity=0.2 -> lower=0.0 upper=0.20 effort=100.0 velocity=0.2; origin xyz=0.008271576273727 0.137279512977855 0.036010455529876 rpy=0 0 0 -> xyz=0.008271576273727 0.137279512977855 0.0435 rpy=0 0 0
