Commit message: auto pick palce 0

File: src/robot0_description/urdf/robot0.urdf (robot description, URDF)
Before this commit: robot robot0, 9 links, 8 joints
Links:
- link base_link: geometry collision box size=0.28 0.24 0.06; visual mesh filename=package://robot0_description/meshes/base_link.stl
- link lift_arm_link: geometry collision box size=0.051 0.149 0.136; collision box size=0.115 0.018 0.004
Joints:
- joint base_footprint_joint: origin xyz=0 0 0.06 rpy=0 0 -1.5707963267948966 -> xyz=0 0 0.06 rpy=0 0 0
- joint camera_joint: origin xyz=0.00767 0.1788 0.272 rpy=0 0.7 1.5707963267948966 -> xyz=0.1788 -0.00767 0.272 rpy=0 0.7 0
- joint lift_arm_joint: origin xyz=0.008271576273727 0.137279512977855 0.0435 rpy=0 0 0 -> xyz=0.137279512977855 -0.008271576273727 0.0435 rpy=0 0 0
- joint wheel_fl_joint: origin xyz=-0.145628423726273 0.109279512977855 -0.02385 rpy=1.5707963267949 -1.5707963267949 0 -> xyz=0.109279512977855 0.145628423726273 -0.02385 rpy=1.5707963267949 -1.5707963267949 -1.5707963267948966
- joint wheel_fr_joint: origin xyz=0.162171576273727 0.109279512977855 -0.02385 rpy=-1.5707963267949 -1.5707963267949 0 -> xyz=0.109279512977855 -0.162171576273727 -0.02385 rpy=-1.5707963267949 -1.5707963267949 -1.5707963267948966
- joint wheel_rl_joint: origin xyz=-0.145628423726273 -0.090720487022145 -0.02385 rpy=1.5707963267949 -1.5707963267949 0 -> xyz=-0.090720487022145 0.145628423726273 -0.02385 rpy=1.5707963267949 -1.5707963267949 -1.5707963267948966
- joint wheel_rr_joint: origin xyz=0.162171576273727 -0.090720487022145 -0.02385 rpy=-1.5707963267949 -1.5707963267949 0 -> xyz=-0.090720487022145 -0.162171576273727 -0.02385 rpy=-1.5707963267949 -1.5707963267949 -1.5707963267948966
