Commit message: fix model 3d

File: src/robot0_description/urdf/camera.xacro (robot description, xacro)
@@ -11,7 +11,7 @@
     </inertial>
   </link>
-  <!-- Joint from base_link to camera_link: forward in +X, tilted down by 0.7 rad pitch -->
+  <!-- Joint from base_link to camera_link: forward in +X, tilted down by camera_pitch -->
   <joint name="camera_joint" type="fixed">
-    <origin xyz="0.1788 -0.00767 0.272" rpy="0 0.7 0" />
+    <origin xyz="${camera_joint_x} ${camera_joint_y} ${camera_joint_z}" rpy="0 ${camera_pitch} 0" />
     <parent link="base_link" />
     <child link="camera_link" />
@@ -20,5 +20,5 @@
   <link name="camera_optical_link" />
   <joint name="camera_optical_joint" type="fixed">
-    <origin xyz="0 0 0" rpy="-1.5707963267948966 0 -1.5707963267948966" />
+    <origin xyz="0 0 0" rpy="-${PI/2} 0 -${PI/2}" />
     <parent link="camera_link" />
     <child link="camera_optical_link" />

File: src/robot0_description/urdf/chassis.xacro (robot description, xacro)
@@ -12,11 +12,11 @@
   <link name="base_link">
     <inertial>
-      <origin xyz="-0.0003708 -0.0082536 0.0149603" rpy="0 0 0" />
+      <origin xyz="-0.00965 0.00000 0.01496" rpy="0 0 0" />
       <mass value="1.85" />
       <inertia ixx="0.010" ixy="0" ixz="0" iyy="0.005" iyz="0" izz="0.012" />
     </inertial>
-    <!-- Main Chassis Base -->
+    <!-- Main Chassis Base (Offset CAD origin to center base_link at 0,0,0) -->
     <visual>
-      <origin xyz="0 0 0" rpy="0 0 0" />
+      <origin xyz="-0.00928 0.00827 0.0" rpy="0 0 0" />
       <geometry>
         <mesh filename="package://robot0_description/meshes/base_link.stl" />
@@ -24,13 +24,14 @@
       <material name="silver" />
     </visual>
+    <!-- Collision Box sized to prevent overlap with front lift carriage -->
     <collision>
-      <origin xyz="0.01 -0.0083 0.03" rpy="0 0 0" />
+      <origin xyz="-0.010 0.000 0.030" rpy="0 0 0" />
       <geometry>
-        <box size="0.28 0.24 0.06" />
+        <box size="0.22 0.24 0.06" />
       </geometry>
     </collision>
     <!-- Front-Right Motor Bracket -->
     <visual>
-      <origin xyz="0.129279512977854 -0.131271576273728 -0.00376593806610101" rpy="-1.5707963267949 0 1.5707963267948934" />
+      <origin xyz="0.120 -0.123 -0.00377" rpy="-${PI/2} 0 ${PI/2}" />
       <geometry>
         <mesh filename="package://robot0_description/meshes/motor_bracket_fr.stl" />
@@ -40,5 +41,5 @@
     <!-- Front-Left Motor Bracket -->
     <visual>
-      <origin xyz="0.089279512977854 0.114728423726273 -0.00376593806610101" rpy="-1.5707963267949 0 -1.5707963267948966" />
+      <origin xyz="0.080 0.123 -0.00377" rpy="-${PI/2} 0 -${PI/2}" />
       <geometry>
         <mesh filename="package://robot0_description/meshes/motor_bracket_fl.stl" />
@@ -48,5 +49,5 @@
     <!-- Rear-Right Motor Bracket -->
     <visual>
-      <origin xyz="-0.070720487022142 -0.131271576273728 -0.003765938066101" rpy="-1.5707963267949 0 1.5707963267948934" />
+      <origin xyz="-0.080 -0.123 -0.00377" rpy="-${PI/2} 0 ${PI/2}" />
       <geometry>
         <mesh filename="package://robot0_description/meshes/motor_bracket_rr.stl" />
@@ -56,5 +57,5 @@
     <!-- Rear-Left Motor Bracket -->
     <visual>
-      <origin xyz="-0.115720487022144 0.114728423726274 -0.00376593806610199" rpy="-1.57079632679489 0 -1.5707963267948966" />
+      <origin xyz="-0.125 0.123 -0.00377" rpy="-${PI/2} 0 -${PI/2}" />
       <geometry>
         <mesh filename="package://robot0_description/meshes/motor_bracket_rl.stl" />
@@ -64,5 +65,5 @@
     <!-- Front-Right Motor -->
     <visual>
-      <origin xyz="0.109279512977855 -0.128271576273727 -0.0307659380661" rpy="1.5707963267949 0 0" />
+      <origin xyz="0.100 -0.120 -0.03077" rpy="${PI/2} 0 0" />
       <geometry>
         <mesh filename="package://robot0_description/meshes/motor_jgb37_520_right.stl" />
@@ -72,5 +73,5 @@
     <!-- Front-Left Motor -->
     <visual>
-      <origin xyz="0.109279512977855 0.111728423726273 -0.0307659380661" rpy="-1.5707963267949 0 -3.141592653589793" />
+      <origin xyz="0.100 0.120 -0.03077" rpy="-${PI/2} 0 -${PI}" />
       <geometry>
         <mesh filename="package://robot0_description/meshes/motor_jgb37_520_left.stl" />
@@ -80,5 +81,5 @@
     <!-- Rear-Right Motor -->
     <visual>
-      <origin xyz="-0.090720487022144 -0.128271576273727 -0.0307659380661" rpy="1.5707963267949 0 0" />
+      <origin xyz="-0.100 -0.120 -0.03077" rpy="${PI/2} 0 0" />
       <geometry>
         <mesh filename="package://robot0_description/meshes/motor_jgb37_520_right.stl" />
@@ -88,5 +89,5 @@
     <!-- Rear-Left Motor -->
     <visual>
-      <origin xyz="-0.090720487022144 0.111728423726273 -0.0307659380661" rpy="-1.5707963267949 0 -3.141592653589793" />
+      <origin xyz="-0.100 0.120 -0.03077" rpy="-${PI/2} 0 -${PI}" />
       <geometry>
         <mesh filename="package://robot0_description/meshes/motor_jgb37_520_left.stl" />
@@ -96,5 +97,5 @@
     <!-- Lift Base Column -->
     <visual>
-      <origin xyz="0.137279512977854 -0.008271576273727 0.00223406193389999" rpy="1.5707963267949 0 -1.5707963267948966" />
+      <origin xyz="0.128 0.000 0.00223" rpy="${PI/2} 0 -${PI/2}" />
       <geometry>
         <mesh filename="package://robot0_description/meshes/lift_base.stl" />
@@ -104,5 +105,5 @@
     <!-- Lift Motor -->
     <visual>
-      <origin xyz="0.119779512977854 -0.008271576273727 0.0292340619339" rpy="-1.5707963267949 0 -1.5707963267948966" />
+      <origin xyz="0.1105 0.000 0.02923" rpy="-${PI/2} 0 -${PI/2}" />
       <geometry>
         <mesh filename="package://robot0_description/meshes/motor_jgb37_520_right.stl" />
@@ -112,5 +113,5 @@
     <!-- Lift Guide Pipe 1 -->
     <visual>
-      <origin xyz="0.137279512977855 -0.065771576273727 0.00823406193389999" rpy="1.5707963267949 0 -3.2923750299165266" />
+      <origin xyz="0.128 -0.0575 0.00823" rpy="${PI/2} 0 -3.292375" />
       <geometry>
         <mesh filename="package://robot0_description/meshes/lift_pipe_1.stl" />
@@ -120,5 +121,5 @@
     <!-- Lift Guide Pipe 2 -->
     <visual>
-      <origin xyz="0.137279512977855 -0.008271576273727 0.046010455529876" rpy="1.5707963267949 0 -2.9908102772630566" />
+      <origin xyz="0.128 0.000 0.04601" rpy="${PI/2} 0 -2.990810" />
       <geometry>
         <mesh filename="package://robot0_description/meshes/lift_pipe_2.stl" />
@@ -128,5 +129,5 @@
     <!-- Lift Top Cap -->
     <visual>
-      <origin xyz="0.137279512977854 -0.008271576273728 0.2682340619339" rpy="1.5707963267949 0 -1.5707963267948966" />
+      <origin xyz="0.128 0.000 0.26823" rpy="${PI/2} 0 -${PI/2}" />
       <geometry>
         <mesh filename="package://robot0_description/meshes/lift_top_cap.stl" />
@@ -136,5 +137,5 @@
     <!-- Lift Timing Belt -->
     <visual>
-      <origin xyz="0.128279512977855 -0.008271576273728 0.2782340619339" rpy="1.5707963267949 1.5707963267949 -1.5707963267948966" />
+      <origin xyz="0.119 0.000 0.27823" rpy="${PI/2} ${PI/2} -${PI/2}" />
       <geometry>
         <mesh filename="package://robot0_description/meshes/lift_belt.stl" />
@@ -144,5 +145,5 @@
     <!-- Lift Top Pulley -->
     <visual>
-      <origin xyz="0.128279512977855 -0.008271576273728 0.2797340619339" rpy="-1.5707963267949 -0.897413987985829 1.5707963267948934" />
+      <origin xyz="0.119 0.000 0.27973" rpy="-${PI/2} -0.897414 ${PI/2}" />
       <geometry>
         <mesh filename="package://robot0_description/meshes/lift_pulley_20t.stl" />

File: src/robot0_description/urdf/common_properties.xacro (robot description, xacro)
@@ -22,6 +22,12 @@
   </material>
   <!-- ========================================== -->
+  <!-- Robot0 Geometric & Kinematic Properties    -->
+  <!-- ========================================== -->
+  <!-- Wheelbase (Front-to-Rear) = 0.200m -> lx = 0.100m -->
+  <xacro:property name="wheelbase_lx" value="0.100" />
+  <!-- Track Width (Left-to-Right) = 0.3078m -> ly = 0.1539m -->
+  <xacro:property name="track_ly" value="0.1539" />
+  <xacro:property name="wheel_z_offset" value="-0.02385" />
   <!-- Wheel Common Properties                    -->
-  <!-- ========================================== -->
   <xacro:property name="wheel_radius" value="0.0487" />
   <xacro:property name="wheel_length" value="0.045" />
@@ -29,3 +35,12 @@
   <xacro:property name="wheel_effort_limit" value="10.0" />
   <xacro:property name="wheel_velocity_limit" value="20.0" />
+  <!-- Lift Mechanism Kinematics -->
+  <xacro:property name="lift_joint_x" value="0.128" />
+  <xacro:property name="lift_joint_y" value="0.000" />
+  <xacro:property name="lift_joint_z" value="0.0435" />
+  <!-- Camera Sensor Kinematics -->
+  <xacro:property name="camera_joint_x" value="0.1695" />
+  <xacro:property name="camera_joint_y" value="0.000" />
+  <xacro:property name="camera_joint_z" value="0.272" />
+  <xacro:property name="camera_pitch" value="0.70" />
 </robot>

File: src/robot0_description/urdf/lift.xacro (robot description, xacro)
@@ -6,10 +6,10 @@
   <link name="lift_arm_link">
     <inertial>
-      <origin xyz="-0.0180613677899576 -3.0454656503736E-05 -0.0256536372783613" rpy="1.5707963267949 0 -1.5707963267948966" />
-      <mass value="0.161814335334686" />
+      <origin xyz="-0.01806 0.00000 -0.02565" rpy="${PI/2} 0 -${PI/2}" />
+      <mass value="0.16181" />
       <inertia ixx="0.00038242" ixy="-1.38e-07" ixz="-1.26e-07" iyy="0.00045993" iyz="-0.00018047" izz="0.00040656" />
     </inertial>
     <visual>
-      <origin xyz="0 0 0" rpy="1.5707963267949 0 -1.5707963267948966" />
+      <origin xyz="0 0 0" rpy="${PI/2} 0 -${PI/2}" />
       <geometry>
         <mesh filename="package://robot0_description/meshes/lift_arm.stl" />
@@ -19,5 +19,5 @@
     <!-- Back Vertical Slider Carriage Collision -->
     <collision name="lift_arm_slider_collision">
-      <origin xyz="0.008 0 -0.048" rpy="0 0 0" />
+      <origin xyz="0.008 0.000 -0.048" rpy="0 0 0" />
       <geometry>
         <box size="0.051 0.149 0.136" />
@@ -55,7 +55,7 @@
     </collision>
   </link>
-  <!-- Prismatic Joint: Moves along Z axis (UP) -->
+  <!-- Prismatic Joint: Moves along Z axis (UP), Centered on Y=0 -->
   <joint name="lift_arm_joint" type="prismatic">
-    <origin xyz="0.137279512977855 -0.008271576273727 0.0435" rpy="0 0 0" />
+    <origin xyz="${lift_joint_x} ${lift_joint_y} ${lift_joint_z}" rpy="0 0 0" />
     <parent link="base_link" />
     <child link="lift_arm_link" />

File: src/robot0_description/urdf/wheel.xacro (robot description, xacro)
@@ -48,6 +48,6 @@
     mesh_type="wheel_right"
     mesh_rpy="${PI} 0 0"
-    joint_xyz="0.109279512977855 -0.162171576273727 -0.02385"
-    joint_rpy="-1.5707963267949 -1.5707963267949 -1.5707963267948966"
+    joint_xyz="${wheelbase_lx} -${track_ly} ${wheel_z_offset}"
+    joint_rpy="-${PI/2} -${PI/2} -${PI/2}"
     axis_xyz="0 -1 0" />
   <!-- Front-Left Wheel -->
@@ -57,6 +57,6 @@
     mesh_type="wheel_left"
     mesh_rpy="0 0 0"
-    joint_xyz="0.109279512977855 0.145628423726273 -0.02385"
-    joint_rpy="1.5707963267949 -1.5707963267949 -1.5707963267948966"
+    joint_xyz="${wheelbase_lx} ${track_ly} ${wheel_z_offset}"
+    joint_rpy="${PI/2} -${PI/2} -${PI/2}"
     axis_xyz="0 1 0" />
   <!-- Rear-Right Wheel -->
@@ -66,6 +66,6 @@
     mesh_type="wheel_left"
     mesh_rpy="${PI} 0 ${PI}"
-    joint_xyz="-0.090720487022145 -0.162171576273727 -0.02385"
-    joint_rpy="-1.5707963267949 -1.5707963267949 -1.5707963267948966"
+    joint_xyz="-${wheelbase_lx} -${track_ly} ${wheel_z_offset}"
+    joint_rpy="-${PI/2} -${PI/2} -${PI/2}"
     axis_xyz="0 -1 0" />
   <!-- Rear-Left Wheel -->
@@ -75,6 +75,6 @@
     mesh_type="wheel_right"
     mesh_rpy="0 0 ${PI}"
-    joint_xyz="-0.090720487022145 0.145628423726273 -0.02385"
-    joint_rpy="1.5707963267949 -1.5707963267949 -1.5707963267948966"
+    joint_xyz="-${wheelbase_lx} ${track_ly} ${wheel_z_offset}"
+    joint_rpy="${PI/2} -${PI/2} -${PI/2}"
     axis_xyz="0 1 0" />
 </robot>
